File: pos-receiver-sch/mainboard/mainboard.sch (EAGLE design)
At the start: 30 parts, among them IC1 TLC274D, Q1 L78M05CDT

Commit message: mainboard
Parts:
- R12: device resistor:R-EU_M0805 -> resistor:R-EU_M1206
- R5: device resistor:R-EU_M0805 -> resistor:R-EU_R1206
Connections:
- removed net N$3: IC1B.-IN, R11.A, R11.S, R12.2
- new net N$2: IC1B.-IN, R11.E, R11.S, R12.2
- net +3V3: now also U$1.VDD; no longer U$1.VDD2
- net +5V: now also U$1.5V2
- net GND: now also U$1.GND1, U$1.GND3, U$1.GND7
- net N$13: now also R11.A; no longer R11.E
- net N$20: now also R8.A; no longer R8.E
- net N$6: now also R8.E; no longer R8.A
Other:
- moved on the sheet: R11, R8
