File: pos-receiver-sch/mainboard/mainboard.brd (EAGLE design)
At the start: 100 x 80 mm, 30 parts, among them IC1 TLC274D, Q1 L78M05CDT

Commit message: mainboard
Parts:
- R12: device resistor:M0805 -> resistor:M1206
- R5: device resistor:M0805 -> resistor:R1206
- moved JP4 56.2 mm to (54.6, 69.8), turned to 180 degrees
- moved C7 25.8 mm to (46.4, 64.8)
- moved R7 25.3 mm to (46.4, 69.2)
- moved C1 24.9 mm to (41.9, 69.2)
- moved R6 24.2 mm to (52.7, 46.4)
- moved JP1 23.3 mm to (63.5, 39.4), turned to 180 degrees
- moved JP2 22.0 mm to (50.2, 39.4), turned to 180 degrees
- moved JP3 21.7 mm to (38.1, 39.4), turned to 180 degrees
- moved C4 20.1 mm to (61.0, 45.7)
- moved R2 19.5 mm to (61.0, 50.2)
- moved R1 17.4 mm to (48.9, 48.9)
- moved C3 17.3 mm to (47.6, 43.8)
- moved R5 13.6 mm to (38.1, 54.0), turned to 180 degrees
- moved R10 13.3 mm to (54.6, 51.4), turned to 270 degrees
- moved R8 12.1 mm to (38.1, 60.3)
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Connections:
- removed net N$3: IC1.6, R11.2, R11.3, R12.2
- new net N$2: IC1.6, R11.1, R11.2, R12.2
- net +3V3: now also U$1.P$3; no longer U$1.P$55
- net +5V: now also U$1.P$54
- net GND: now also U$1.P$2, U$1.P$23, U$1.P$52
- net N$13: now also R11.3; no longer R11.1
- net N$20: now also R8.3; no longer R8.1
- net N$6: now also R8.1; no longer R8.3
Routing:
- net GND: track 0.00 -> 284.9 mm
- net +12V: track 0.00 -> 97.6 mm
- net PA4: track 0.00 -> 62.9 mm
- net +3V3: track 0.00 -> 43.5 mm
- net N$16: track 0.00 -> 39.8 mm
- net PC5: track 0.00 -> 24.2 mm
- net N$13: track 0.00 -> 24.1 mm
- net N$20: track 0.00 -> 21.2 mm
- net PA1: track 0.00 -> 14.1 mm
- net N$4: track 0.00 -> 14.0 mm
- net N$19: track 0.00 -> 13.7 mm
- net N$2: track 0.00 -> 13.6 mm
- net N$1: track 0.00 -> 10.3 mm
- net +5V: track 0.00 -> 9.35 mm
- net PC4: track 0.00 -> 8.50 mm
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Other:
- board text added: "+"
- board text added: "-"
- board text added: "stawel"
- board text added: "v0.1 receiver mainboard"

Commit message: mainboard
Routing:
- net N$3: track 0.00 -> 213.4 mm
Changed lines of the file:
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@@
 <wire x1="59.68" y1="55.245" x2="59.785" y2="55.35" width="0.4064" layer="1"/>
+</signal>
+<signal name="N$3">
+<wire x1="25.4" y1="29.845" x2="25.4" y2="33.02" width="0" layer="19" extent="1-16"/>
+<wire x1="25.4" y1="33.02" x2="25.4" y2="76.2" width="0.254" layer="1"/>
+<wire x1="25.4" y1="76.2" x2="88.9" y2="76.2" width="0.254" layer="1"/>
+<wire x1="88.9" y1="76.2" x2="88.9" y2="33.02" width="0.254" layer="1"/>
+<wire x1="88.9" y1="33.02" x2="25.4" y2="33.02" width="0.254" layer="1"/>
 </signal>
 </signals>
