File: pos-receiver-sch/receiver/receiver.brd (EAGLE design)
At the start: 100 x 80 mm, 17 parts, among them IC1 AD8599R

Commit message: zmiany w schemacie
Parts:
- C1: value (none) -> 10n
- C2: value (none) -> 22p
- C3, C4, C6, C7: value (none) -> 100n
- C5: value (none) -> 10u
- R1, R4, R6, R7: value (none) -> 10k
- R2: value (none) -> 200k
- R3, R5: value (none) -> 3.3k
Changed lines of the file:
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@@
 <attribute name="OC_FARNELL" value="1438872" x="66.675" y="0.635" size="1.778" layer="27" display="off"/>
 </element>
-<element name="R1" library="resistor" package="R0805" value="" x="45.72" y="13.97"/>
-<element name="R2" library="resistor" package="R0805" value="" x="53.34" y="23.495" rot="R90"/>
-<element name="R3" library="resistor" package="R0805" value="" x="50.8" y="15.24"/>
-<element name="R4" library="resistor" package="R0805" value="" x="49.53" y="30.48" rot="R180"/>
-<element name="R5" library="resistor" package="R0805" value="" x="43.18" y="23.495" rot="R90"/>
-<element name="R6" library="resistor" package="R0805" value="" x="53.34" y="27.94" rot="R90"/>
-<element name="R7" library="resistor" package="R0805" value="" x="57.15" y="26.67" rot="R180"/>
-<element name="C1" library="resistor" package="C1206K" value="" x="54.2925" y="15.5575" rot="R90"/>
-<element name="C2" library="resistor" package="C1206K" value="" x="45.72" y="16.51"/>
-<element name="C3" library="resistor" package="C1206K" value="" x="41.275" y="18.7325" rot="R90"/>
-<element name="C4" library="resistor" package="C1206K" value="" x="56.515" y="22.86" rot="R270"/>
-<element name="C5" library="resistor" package="C1206K" value="" x="57.15" y="29.21"/>
+<element name="R1" library="resistor" package="R0805" value="10k" x="45.72" y="13.97"/>
+<element name="R2" library="resistor" package="R0805" value="200k" x="53.34" y="23.495" rot="R90"/>
+<element name="R3" library="resistor" package="R0805" value="3.3k" x="50.8" y="15.24"/>
+<element name="R4" library="resistor" package="R0805" value="10k" x="49.53" y="30.48" rot="R180"/>
+<element name="R5" library="resistor" package="R0805" value="3.3k" x="43.18" y="23.495" rot="R90"/>
+<element name="R6" library="resistor" package="R0805" value="10k" x="53.34" y="27.94" rot="R90"/>
+<element name="R7" library="resistor" package="R0805" value="10k" x="57.15" y="26.67" rot="R180"/>
+<element name="C1" library="resistor" package="C1206K" value="10n" x="54.2925" y="15.5575" rot="R90"/>
+<element name="C2" library="resistor" package="C1206K" value="22p" x="45.72" y="16.51"/>
+<element name="C3" library="resistor" package="C1206K" value="100n" x="41.275" y="18.7325" rot="R90"/>
+<element name="C4" library="resistor" package="C1206K" value="100n" x="56.515" y="22.86" rot="R270"/>
+<element name="C5" library="resistor" package="C1206K" value="10u" x="57.15" y="29.21"/>
 <element name="JP1" library="pinhead" package="1X03" value="" x="48.26" y="34.29"/>
-<element name="C6" library="resistor" package="C1206" value="" x="57.15" y="31.75"/>
-<element name="C7" library="resistor" package="C1206" value="" x="46.99" y="27.94" rot="R180"/>
+<element name="C6" library="resistor" package="C1206" value="100n" x="57.15" y="31.75"/>
+<element name="C7" library="resistor" package="C1206" value="100n" x="46.99" y="27.94" rot="R180"/>
 <element name="SP1" library="buzzer" package="AL201P" value="AL201P" x="49.2125" y="19.685" rot="R180">
 <attribute name="OC_NEWARK" value="unknown" x="49.2125" y="19.685" size="1.778" layer="27" rot="R180" display="off"/>

Commit message: receiver-sch ver: 0.2
Parts:
- added C8: 100p, resistor:C1206K
- added IC2: 78L10F, linear:SOT89
- C2: value 22p -> 100p
- R1, R4: value 10k -> 33k
- moved C6 11.7 mm to (45.4, 31.8), turned to 180 degrees
- moved C5 10.6 mm to (49.8, 36.8), turned to 270 degrees
- moved JP1 9.09 mm to (40.0, 30.5), turned to 90 degrees
- moved R4 4.86 mm to (54.3, 29.5), turned to 90 degrees
- moved R6 4.72 mm to (56.5, 31.4)
- moved R5 1.00 mm to (42.2, 23.8), turned to 0 degrees
- moved R7 1.00 mm to (57.5, 27.6)
Connections:
- new net N$10: C5.1, IC2.3, JP1.2
- net GND: now also IC2.2, IC2.2@1
- net N$4: now also C8.1
- net N$5: now also C8.2
- net VCC: now also IC2.1; no longer C5.1, JP1.2
Routing:
- net N$10: track 0.00 -> 24.9 mm
- net GND: track 33.5 -> 47.9 mm
- net N$5: track 6.12 -> 11.2 mm
- net N$2: track 9.61 -> 11.3 mm
- net VCC: track 23.4 -> 24.4 mm
- net N$7: track 11.9 -> 12.9 mm
- net N$4: track 15.0 -> 15.9 mm
- net N$1: track 6.41 -> 5.59 mm
- net N$8: track 10.5 -> 11.3 mm
- net N$3: track 3.13 -> 3.82 mm

Commit message: charge amp
Parts:
- removed C1: 10n, resistor:C1206K
- removed IC2: 78L10F, linear:SOT89
- removed R2: 200k, resistor:R0805
- removed R3: 3.3k, resistor:R0805
- C7: device resistor:C1206 -> resistor:C1206K
- moved R7 21.2 mm to (36.8, 22.9)
- moved R4 20.2 mm to (34.9, 35.2)
- moved C4 19.8 mm to (36.8, 20.3), turned to 0 degrees
- moved SP1 17.0 mm to (34.0, 27.3), turned to 0 degrees
- moved R1 16.6 mm to (31.8, 22.9)
- moved C5 16.5 mm to (40.6, 23.2)
- moved IC1 16.2 mm to (34.3, 29.2)
- moved C3 15.9 mm to (26.7, 25.1)
- moved C8 15.3 mm to (37.8, 35.6)
- moved R6 15.0 mm to (41.9, 27.9), turned to 0 degrees
- moved R5 14.9 mm to (28.9, 30.5)
- moved C2 14.5 mm to (31.8, 20.3)
- moved C7 9.72 mm to (41.0, 35.6), turned to 270 degrees
- moved C6 8.78 mm to (43.5, 23.2), turned to 270 degrees
- moved JP1 7.67 mm to (47.0, 27.3), turned to 270 degrees
Connections:
- removed net N$10: C5.1, IC2.3, JP1.2
- removed net N$2: C2.2, IC1.2, R1.2, R3.1
- removed net N$7: IC1.3, R2.1, SP1.2
- net GND: no longer C1.2, IC2.2, IC2.2@1, SP1.1
- net N$3: now also C2.2, IC1.2, R1.2, SP1.1; no longer C1.1, R3.2
- net N$9: now also IC1.3, SP1.2; no longer R2.2
- net VCC: now also C5.1, JP1.2; no longer IC2.1
Routing:
- net GND: track 47.9 -> 18.1 mm
- net N$10: track 24.9 -> 0.00 mm
- net VCC: track 24.4 -> 45.0 mm
- net N$7: track 12.9 -> 0.00 mm
- net N$2: track 11.3 -> 0.00 mm
- net N$3: track 3.82 -> 13.2 mm
- net N$9: track 12.2 -> 21.4 mm
- net N$1: track 5.59 -> 10.0 mm
- net N$4: track 15.9 -> 12.9 mm
- net N$5: track 11.2 -> 12.8 mm
- net N$8: track 11.3 -> 12.4 mm
- net N$6: track 3.62 -> 4.53 mm
Other:
- board text removed: "stawel"

Commit message: pcb
Parts:
- moved C7 4.72 mm to (42.5, 31.1), turned to 0 degrees
- moved C3 1.62 mm to (27.0, 23.5)
- moved C8 1.42 mm to (39.1, 34.9), turned to 0 degrees
- moved R5 0.95 mm to (28.9, 31.4)
- moved C2 0.71 mm to (31.1, 20.6)
- moved R4 0.71 mm to (34.3, 34.9), turned to 180 degrees
- moved R1 0.64 mm to (31.8, 23.5)
- moved R7 0.64 mm to (36.8, 23.5)
- moved C4 0.32 mm to (36.8, 20.6)
Routing:
- net VCC: track 45.0 -> 37.4 mm
- net N$1: track 10.0 -> 3.47 mm
- net N$5: track 12.8 -> 17.5 mm
- net N$6: track 4.53 -> 6.93 mm
- net N$9: track 21.4 -> 19.2 mm
- net N$8: track 12.4 -> 10.3 mm
- net N$3: track 13.2 -> 12.0 mm
Other:
- board size 100 x 80 mm -> 26 x 21.9 mm
- board text added: "stawel"
- board text added: "ver:0.3"

Commit message: pcb
Parts:
- C2: value 100p -> 12p; device resistor:C1206K -> resistor:C0805
- C3, C4, C5, C8: device resistor:C1206K -> resistor:C0805
- IC1: value AD8599R -> NE5532D; device analog-devices:SO8 -> linear:SO08
- R1: value 33k -> 1M
- moved R6 2.69 mm to (40.0, 29.8)
- moved C3 2.01 mm to (28.9, 22.9)
- moved JP1 1.91 mm to (45.1, 27.3)
- moved C7 1.85 mm to (41.0, 32.1)
- moved C6 1.62 mm to (41.9, 23.5)
- moved C2 1.59 mm to (32.1, 21.9)
- moved C4 1.42 mm to (36.2, 21.9)
- moved C5 1.31 mm to (39.4, 22.9)
- moved C8 0.90 mm to (38.4, 34.3)
- moved R7 0.90 mm to (36.2, 24.1)
- moved R5 0.71 mm to (29.5, 31.1)
- moved R1 0.71 mm to (32.1, 24.1)
- moved R4 0.63 mm to (34.3, 34.3)
Routing:
- net VCC: track 37.4 -> 31.6 mm
- net N$5: track 17.5 -> 14.3 mm
- net N$8: track 10.3 -> 7.55 mm
- net GND: track 18.2 -> 15.5 mm
- net N$9: track 19.2 -> 16.6 mm
- net N$6: track 6.93 -> 8.37 mm
- net N$3: track 12.0 -> 10.6 mm
- net N$4: track 13.2 -> 12.0 mm
Other:
- board size 26 x 21.9 mm -> 23.2 x 20.6 mm
- board text added: "rev:4"
- board text removed: "ver:0.3"
